File: hardware/astra_radio/astra_radio.kicad_sch (KiCad schematic)
At the start: 0 parts

Commit message: Lots of new stuff, but lost some stuff :-)
Other:
- added sheet Sensing - RF (sensing_rf.kicad_sch)
- sheet Connectors ports: added {UART0}, {UART1}, {USB}; removed none
- sheet MCU - IO ports: added {UART1}, {USB}; removed none
Changed lines of the file:
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@@
 	(generator_version "10.0")
 	(paper "A4")
-	(hierarchical_label "LNA_IN"
-		(shape input)
-		(at 96.52 59.69 0)
-		(effects
-			(font
-				(size 1.27 1.27)
-			)
-			(justify left)
+	(bus
+		(pts
+			(xy 41.91 63.5) (xy 96.52 63.5)
+		)
+		(stroke
+			(width 0)
+			(type default)
+		)
+	)
+	(bus
+		(pts
+			(xy 41.91 67.31) (xy 96.52 67.31)
+		)
+		(stroke
+			(width 0)
+			(type default)
+		)
+	)
+	(bus
+		(pts
+			(xy 41.91 71.12) (xy 96.52 71.12)
+		)
+		(stroke
+			(width 0)
+			(type default)
 		)
 	)
@@
 		)
 		(fill
-			(color 0 194 194 1)
+			(color 0 194 0 1)
 		)
 		(property "Sheetname" "MCU - Power"
@@
 		)
 		(fill
-			(color 0 194 194 1)
+			(color 0 194 0 1)
 		)
 		(property "Sheetname" "MCU - IO"
@@
 		)
 		(pin "{UART0}" bidirectional
+			(at 96.52 71.12 180)
+			(effects
+				(font
+					(size 1.27 1.27)
+					(color 0 0 0 1)
+				)
+				(justify left)
+			)
+		)
+		(pin "{UART1}" bidirectional
+			(at 96.52 67.31 180)
+			(effects
+				(font
+					(size 1.27 1.27)
+				)
+				(justify left)
+			)
+		)
+		(pin "{USB}" bidirectional
 			(at 96.52 63.5 180)
 			(effects
 				(font
 					(size 1.27 1.27)
-					(color 0 0 0 1)
 				)
 				(justify left)
@@
 	)
 	(sheet
-		(at 58.42 26.67)
+		(at 53.34 81.28)
+		(size 20.32 12.7)
+		(exclude_from_sim no)
+		(in_bom yes)
+		(on_board yes)
+		(dnp no)
+		(fields_autoplaced yes)
+		(stroke
+			(width 0.1524)
+			(type solid)
+		)
+		(fill
+			(color 0 255 255 1)
+		)
+		(property "Sheetname" "Sensing - RF"
+			(at 53.34 80.5684 0)
+			(show_name no)
+			(do_not_autoplace no)
+			(effects
+				(font
+					(size 1.27 1.27)
+				)
+				(justify left bottom)
+			)
+		)
+		(property "Sheetfile" "sensing_rf.kicad_sch"
+			(at 53.34 94.5646 0)
+			(show_name no)
+			(do_not_autoplace no)
+			(effects
+				(font
+					(size 1.27 1.27)
+				)
+				(justify left top)
+			)
+		)
+		(instances
+			(project "astra_radio"
+				(path "/8884176c-0d80-4e55-a09d-e5f02dc9ed2c"
+					(page "6")
+				)
+			)
+		)
+	)
+	(sheet
+		(at 53.34 40.64)
 		(size 25.4 17.78)
 		(exclude_from_sim no)
@@
 		)
 		(property "Sheetname" "Power - Generation"
-			(at 58.42 25.9584 0)
+			(at 53.34 39.9284 0)
 			(show_name no)
 			(do_not_autoplace no)
@@
 		)
 		(property "Sheetfile" "power_generation.kicad_sch"
-			(at 58.42 45.0346 0)
+			(at 53.34 59.0046 0)
 			(show_name no)
 			(do_not_autoplace no)
@@
 	)
 	(sheet
-		(at 18.415 26.67)
+		(at 17.145 55.88)
 		(size 25.4 17.78)
 		(exclude_from_sim no)
@@
 		)
 		(property "Sheetname" "Connectors"
-			(at 18.415 25.9584 0)
+			(at 17.145 55.1684 0)
 			(show_name no)
 			(do_not_autoplace no)
@@
 		)
 		(property "Sheetfile" "connectors.kicad_sch"
-			(at 18.415 45.0346 0)
-			(show_name no)
-			(do_not_autoplace no)
-			(effects
-				(font
-					(size 1.27 1.27)
-				)
-				(justify left top)
-			)
-		)
+			(at 17.145 74.2446 0)
+			(show_name no)
+			(do_not_autoplace no)
+			(effects
+				(font
+					(size 1.27 1.27)
+				)
+				(justify left top)
+			)
+		)
+		(pin "{UART0}" bidirectional
+			(at 42.545 71.12 0)
+			(effects
+				(font
+					(size 1.27 1.27)
+				)
+				(justify right)
+			)
+		)
+		(pin "{UART1}" bidirectional
+			(at 42.545 67.31 0)
+			(effects
+				(font
+					(size 1.27 1.27)
+				)
+				(justify right)
+			)
+		)
+		(pin "{USB}" bidirectional
+			(at 42.545 63.5 0)
+			(effects
+				(font
+					(size 1.27 1.27)
+				)
+				(justify right)
+			)
+		)
