File: hardware/astra_radio/mcu_power.kicad_sch (KiCad schematic)
At the start: 10 parts, among them U2 ESP32-C3

Commit message: Lots of new stuff, but lost some stuff :-)
Parts:
- C10, C12, C7: value 0.1u X7R ??V -> C; footprint Capacitor_SMD:C_0603_1608Metric -> (none)
- C13, C5, C6: value 1u X7R ??V -> C; footprint Capacitor_SMD:C_0603_1608Metric -> (none)
- C3: value 10n X7R ??V -> C; footprint Capacitor_SMD:C_0603_1608Metric -> (none)
- C8: value 10u X7R ??V -> C; footprint Capacitor_SMD:C_0603_1608Metric -> (none)
- L2: value 2.0nH -> L
- U2: footprint Package_DFN_QFN:QFN-32-1EP_5x5mm_P0.5mm_EP3.7x3.7mm -> Package_DFN_QFN:QFN-32-1EP_5x5mm_P0.5mm_EP3.7x3.7mm_ThermalVias; symbol astra_parts:ESP32-C3 - Power -> astra_parts:ESP32-C3_-_Power
