File: hardware/astra_radio/mcu_power.kicad_sch (KiCad schematic)
At the start: 10 parts, among them U2 ESP32-C3

Commit message: Updates to radio
Parts:
- C10, C12, C7: value C -> 0.1uF
- C13: value C -> 10nF
- C3, C5, C6: value C -> 1uF
- C8: value C -> 10uF
- L2: value L -> 2.0nH
Changed lines of the file:
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@@
 			)
 		)
-		(property "Value" "C"
+		(property "Value" "10nF"
 			(at 205.105 91.44 0)
 			(show_name no)
@@
 			)
 		)
-		(property "Value" "C"
+		(property "Value" "0.1uF"
 			(at 128.905 74.93 0)
 			(show_name no)
@@
 			)
 		)
-		(property "Value" "C"
+		(property "Value" "0.1uF"
 			(at 205.105 74.93 0)
 			(show_name no)
@@
 			)
 		)
-		(property "Value" "C"
+		(property "Value" "1uF"
 			(at 149.225 74.93 0)
 			(show_name no)
@@
 			)
 		)
-		(property "Value" "C"
+		(property "Value" "10uF"
 			(at 108.585 74.93 0)
 			(show_name no)
@@
 			)
 		)
-		(property "Value" "C"
+		(property "Value" "0.1uF"
 			(at 149.225 107.95 0)
 			(show_name no)
@@
 			)
 		)
-		(property "Value" "L"
+		(property "Value" "2.0nH"
 			(at 138.43 64.77 90)
 			(show_name no)
@@
 			)
 		)
-		(property "Value" "C"
+		(property "Value" "1uF"
 			(at 156.845 92.71 0)
 			(show_name no)
@@
 			)
 		)
-		(property "Value" "C"
+		(property "Value" "1uF"
 			(at 222.885 91.44 0)
 			(show_name no)
