File: hardware/astra_radio/connectors.kicad_sch (KiCad schematic)
At the start: 8 parts, among them J1 JST_SM04B-GHS-TB, J2 JST_SM06B-GHS-TB, J3 USB_C_Receptacle_USB2.0_16P

Commit message: Updates to radio
Parts:
- added D1, D2, D3: SS23, Diode_SMD:D_SMA, symbol Diode:SS23
Connections:
- net +5V: now also D1.1 (K), D2.1 (K), D3.1 (K); no longer J1.1, J2.1, J3.A4 (VBUS), J3.A9 (VBUS), J3.B4 (VBUS), J3.B9 (VBUS)
- new net: D1.2 (A), J1.1
- new net: D3.2 (A), J3.A4 (VBUS), J3.A9 (VBUS), J3.B4 (VBUS), J3.B9 (VBUS)
- new net: D2.2 (A), J2.1
Other:
- moved on the sheet: C19, C20, C21
