File: hardware/astra_radio/mcu_io.kicad_sch (KiCad schematic)
At the start: 13 parts, among them SW1 SW_SPDT, U1 ESP32-C3, Y1 FW400WFMR1

Commit message: Updates
Connections:
- net U0RXD: no longer U1.27 (U0RXD)
- net U0TXD: no longer R7.1
- new net UART0_RX: U1.27 (U0RXD)
- new net UART0_TX: R7.1

Commit message: Lots of new stuff, but lost some stuff :-)
Parts:
- added AE2: Antenna_Dipole, symbol Device:Antenna_Dipole
- added C14, C15: C, symbol Device:C
- added L3: L, symbol Device:L
- added R10, R11, R12, R13, R9: 499, symbol Device:R
- added R15: R, symbol Device:R
- added TP3, TP4, TP5, TP6: TestPoint, symbol Connector:TestPoint
- C1: value 1u -> C; footprint Capacitor_SMD:C_0603_1608Metric -> (none)
- C11, C9: value 14p -> C; footprint Capacitor_SMD:C_0402_1005Metric -> (none)
- L1: value 24nH -> L
- R1: value 10k -> R; footprint Resistor_SMD:R_0402_1005Metric -> (none)
- R5, R6: value 10K -> R
- SW1: footprint Button_Switch_SMD:SW_SPDT_PCM12 -> (none)
- U1: footprint Package_DFN_QFN:QFN-32-1EP_5x5mm_P0.5mm_EP3.7x3.7mm -> Package_DFN_QFN:QFN-32-1EP_5x5mm_P0.5mm_EP3.7x3.7mm_ThermalVias; symbol astra_parts:ESP32-C3 - IO -> astra_parts:ESP32-C3_-_IO
Connections:
- net +3V3: now also C1.1, R6.2, R15.1
- net Earth: now also AE2.1, C14.2, C15.2
- net GPIO2: now also R15.2; no longer R5.2, U1.14 (GPIO8)
- net LNA_IN: now also C15.1, L3.2
- net U0RXD: now also U1.27 (U0RXD), R10.1; no longer TP1.1
- net U0TXD: now also U1.28 (U0TXD), R11.2; no longer TP2.1
- net UART0_RX: now also TP1.1, R10.2; no longer U1.27 (U0RXD)
- net UART0_TX: now also TP2.1, R11.1; no longer R7.1
- net UART1_TX: now reaches R7.2
- net UART1_TX: now also TP4.1; no longer U1.28 (U0TXD)
- net GPIO0: no longer names the net of U1.5 (XTAL_32K_N)
- net GPIO1: no longer names the net of U1.4 (XTAL_32K_P)
- net GPIO18 renamed USB_D-
- net GPIO19 renamed USB_D+
- net GPIO3 renamed 3V3_PG
- net GPIO4 renamed U1TXD
- net U1TXD: now also R7.1
- net GPIO5 renamed U1RXD
- net U1RXD: now also R9.2
- net GPIO6 renamed U1CTS
- net U1CTS: now also R13.1
- net GPIO7 renamed U1RTS
- net U1RTS: now also R12.2
- new net: AE2.2, C14.1, L3.1
- new net GPIO8: R5.2, U1.14 (GPIO8)
- new net UART1_CTS: R13.2, TP5.1
- new net UART1_RTS: R12.1, TP6.1
- new net UART1_RX: R9.1, TP3.1
- no-connect marks 6 -> 8
Other:
- note added: "Antenna Input"
- note added: "Comms UART"
- note added: "Debug UART"
- note added: "Debug USB"
- note added: "UART1"
- note removed: "LNA IN"
- moved on the sheet: TP1, TP2, U1

Commit message: Alsmot there
Parts:
- C1: value C -> 1u
- R1, R15, R5, R6: value R -> 10K
Changed lines of the file:
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@@
 			)
 		)
-		(property "Value" "R"
+		(property "Value" "10K"
 			(at 166.37 20.32 90)
 			(show_name no)
@@
 			)
 		)
-		(property "Value" "R"
+		(property "Value" "10K"
 			(at 119.38 26.6699 0)
 			(show_name no)
@@
 			)
 		)
-		(property "Value" "C"
+		(property "Value" "1u"
 			(at 175.895 33.02 0)
 			(show_name no)
@@
 			)
 		)
-		(property "Value" "R"
-			(at 106.68 43.18 90)
+		(property "Value" "10K"
+			(at 106.68 40.894 90)
 			(show_name no)
 			(do_not_autoplace no)
@@
 			)
 		)
-		(property "Value" "R"
+		(property "Value" "10K"
 			(at 111.76 26.6699 0)
 			(show_name no)
