File: hardware/astra_radio/mcu_io.kicad_sch (KiCad schematic)
At the start: 27 parts, among them SW1 SW_SPDT, U1 ESP32-C3, Y1 FW400WFMR1

Commit message: Updates to radio
Parts:
- Y1: footprint FW400WFMR1 -> astra_parts:FW400WFMR1
Changed lines of the file:
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@@
 			)
 		)
-		(property "Footprint" "FW400WFMR1"
+		(property "Footprint" "astra_parts:FW400WFMR1"
 			(at 248.92 127.94 0)
 			(hide yes)
