File: hardware/astra_radio/power_generation.kicad_sch (KiCad schematic)
At the start: 0 parts

Commit message: Lots of new stuff, but lost some stuff :-)
Parts:
- added C16, C4: C, symbol Device:C
- added R8: R, symbol Device:R
- added U3: LD39100PU33RY, astra_parts:LD39100PU33RY, symbol astra_parts:LD39100PU33RY
Connections:
- new net +3V3: C16.1, R8.1, U3.4 (VOUT)
- new net +5V: C4.1, U3.1 (EN), U3.6 (VIN)
- new net 3V3_PG: R8.2, U3.3 (PG)
- new net Earth: C16.2, C4.2, U3.2 (GND), U3.7 (EP)

Commit message: Alsmot there
Parts:
- C16, C4: value C -> 1u
- R8: value R -> 100K
Changed lines of the file:
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@@
+	(wire
+		(pts
+			(xy 162.56 97.79) (xy 162.56 101.6)
+		)
+		(stroke
+			(width 0)
+			(type default)
+		)
+	)
 	(wire
 		(pts
@@
 	(wire
 		(pts
-			(xy 162.56 101.6) (xy 175.26 101.6)
+			(xy 162.56 101.6) (xy 173.99 101.6)
 		)
 		(stroke
@@
 	(wire
 		(pts
-			(xy 162.56 97.79) (xy 162.56 101.6)
-		)
-		(stroke
-			(width 0)
-			(type default)
-		)
-	)
-	(wire
-		(pts
 			(xy 171.45 83.82) (xy 171.45 86.36)
 		)
@@
 	)
 	(label "3V3_PG"
-		(at 175.26 101.6 180)
+		(at 173.99 101.6 180)
 		(effects
 			(font
 				(size 1.27 1.27)
+				(color 132 0 0 1)
 			)
 			(justify right bottom)
@@
 		(dnp no)
 		(property "Reference" "C4"
-			(at 123.825 87.63 0)
+			(at 124.206 92.964 0)
 			(show_name no)
 			(do_not_autoplace no)
@@
 			)
 		)
-		(property "Value" "C"
-			(at 123.825 92.71 0)
-			(show_name no)
-			(do_not_autoplace no)
+		(property "Value" "1u"
+			(at 120.65 92.964 0)
+			(show_name no)
+			(do_not_autoplace yes)
 			(effects
 				(font
@@
 			)
 		)
-		(property "Value" "C"
+		(property "Value" "1u"
 			(at 172.085 92.71 0)
 			(show_name no)
@@
 		(in_pos_files yes)
 		(dnp no)
-		(fields_autoplaced yes)
 		(property "Reference" "R8"
-			(at 165.1 92.7099 0)
+			(at 164.338 92.71 0)
 			(show_name no)
 			(do_not_autoplace no)
@@
 			)
 		)
-		(property "Value" "R"
-			(at 165.1 95.2499 0)
-			(show_name no)
-			(do_not_autoplace no)
+		(property "Value" "100K"
+			(at 164.592 94.996 0)
+			(show_name no)
+			(do_not_autoplace no)
